Commit message: Add gripper

File: ros2_packages/robots_adapters/urdf/fr3_gz.urdf.xacro (robot description, xacro)
@@ -3,5 +3,5 @@
   <xacro:arg name="arm_prefix"      default="" />
   <xacro:arg name="robot_namespace" default="" />
-  <xacro:arg name="controllers_file" default="" />   <!-- add this -->
+  <xacro:arg name="controllers_file" default="" />
   <!--
     ros2_control:=false  → skip upstream's broken gz_ros2_control block
@@ -69,6 +69,21 @@
     </joint>
     <joint name="$(arg arm_prefix)_fr3_finger_joint1">
-      <command_interface name="position"/>
-      <state_interface name="position"><param name="initial_value">0.0</param></state_interface>
+      <command_interface name="position">
+        <param name="min">0.0</param>
+        <param name="max">0.04</param>
+      </command_interface>
+      <state_interface name="position">
+        <param name="initial_value">0.04</param>
+      </state_interface>
+      <state_interface name="velocity"/>
+    </joint>
+    <joint name="$(arg arm_prefix)_fr3_finger_joint2">
+      <command_interface name="position">
+        <param name="min">0.0</param>
+        <param name="max">0.04</param>
+      </command_interface>
+      <state_interface name="position">
+        <param name="initial_value">0.04</param>
+      </state_interface>
       <state_interface name="velocity"/>
     </joint>

Commit message: fix the robot to not fall

File: ros2_packages/robots_adapters/urdf/fr3_gz.urdf.xacro (robot description, xacro)
@@ -5,4 +5,5 @@
   <xacro:arg name="controllers_file" default="" />
   <!--
+    Franka description — includes base, link0..7, hand, fingers.
     ros2_control:=false  → skip upstream's broken gz_ros2_control block
     gazebo:=false        → skip ROS1 transmissions
@@ -10,4 +11,39 @@
   -->
   <xacro:include filename="$(find franka_description)/robots/fr3/fr3.urdf.xacro"/>
+  <!--
+    Anchor the robot base to the world in Ignition Fortress.
+    The only approach that works for dynamically spawned robots is to give
+    the base links enormous inertia. With mass=100000kg, any reaction force
+    F from joint motion produces acceleration a = F/m ≈ 0, so the base
+    stays put while all arm joints move normally.
+    Applied to BOTH base and fr3_link0 because:
+      - 'base' is the visual/collision root link
+      - 'fr3_link0' is connected to base via a fixed joint and is the
+        actual physics anchor point that receives joint reaction forces
+        from fr3_joint1
+    gravity=false prevents the huge mass from generating enormous
+    gravitational forces that would crush the physics solver.
+  -->
+  <gazebo reference="base">
+    <gravity>false</gravity>
+    <inertial>
+      <mass>100000</mass>
+      <inertia>
+        <ixx>100000</ixx><iyy>100000</iyy><izz>100000</izz>
+        <ixy>0</ixy><ixz>0</ixz><iyz>0</iyz>
+      </inertia>
+    </inertial>
+  </gazebo>
+  <gazebo reference="$(arg arm_prefix)_fr3_link0">
+    <gravity>false</gravity>
+    <inertial>
+      <mass>100000</mass>
+      <inertia>
+        <ixx>100000</ixx><iyy>100000</iyy><izz>100000</izz>
+        <ixy>0</ixy><ixz>0</ixz><iyz>0</iyz>
+      </inertia>
+    </inertial>
+  </gazebo>
+  <!-- Gazebo plugins, ros2_control, etc. -->
   <!-- ── Correct plugin for Ignition Fortress ─────────────────────────── -->
   <gazebo>
